File: hardware/overlay64.sch (KiCad schematic (older format))
At the start: 26 parts, among them IC1 ATMEGA1284, P1 USB, P2 INPUT, P3 CONTROL, P4 MAIN, P5 HOLE, P6 HOLE, P7 HOLE, P8 HOLE, P9 BYPASS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

Commit message: SMD rework
Parts:
- removed IC1: ATMEGA1284, Housings_DIP:DIP-40_W15.24mm, symbol ATMEGA1284-P
- removed P1: USB, custom:USB-MINI-B-TH, symbol CONN_01X05
- removed SW1: SW_BOOT, custom:Button, symbol SW_PUSH_SMALL_H
- added IC1: ATmega1284P-AU, Package_QFP:TQFP-44_10x10mm_P0.8mm, symbol MCU_Microchip_ATmega:ATmega1284P-AU
- added J: USB_B_Mini, Connector_USB:USB_Mini-B_Lumberg_2486_01_Horizontal, symbol Connector:USB_B_Mini
- C1, C4, C5, C6: symbol C -> Device:C
- C2, C3: symbol C_Small -> Device:C_Small
- D1, D2: symbol ZENER -> overlay64-rescue:ZENER
- P2, P9: symbol CONN_01X16 -> overlay64-rescue:CONN_01X16
- P3: symbol CONN_01X08 -> overlay64-rescue:CONN_01X08
- P4: symbol CONN_01X03 -> overlay64-rescue:CONN_01X03
- P5, P6, P7, P8: symbol CONN_01X01 -> overlay64-rescue:CONN_01X01
- R1, R2, R3, R5: symbol R -> Device:R
- RV1: symbol POT-RESCUE-overlay64 -> overlay64-rescue:POT-RESCUE-overlay64
- U1: symbol LM1881 -> lm1881:LM1881
- Y1: symbol Crystal_Small -> Device:Crystal_Small
Connections:
- wire segments 25 -> 40
- no-connect marks 7 -> 2
Other:
- moved on the sheet: D1, D2, P2, P9
